File: board/pd_board.sch (KiCad schematic (older format))
At the start: 9 parts, among them P1 Vin Gnd, P2 CONN_2, P3 CONN_2, P4 CONN_2, P5 CONN_2, P6 CONN_2, P7 CONN_2, P8 CONN_2, P9 CONN_2

Commit message: Cleanup. Minor changes
Changed lines of the file:
@@
 Sheet 1 1
 Title ""
-Date "14 apr 2014"
+Date "15 apr 2014"
 Rev ""
 Comp ""
@@
 L VCC #PWR016
 U 1 1 534C1618
-P 3100 3250
-F 0 "#PWR016" H 3100 3350 30  0001 C CNN
-F 1 "VCC" H 3100 3350 30  0000 C CNN
-F 2 "" H 3100 3250 60  0000 C CNN
-F 3 "" H 3100 3250 60  0000 C CNN
-	1    3100 3250
+P 3100 3200
+F 0 "#PWR016" H 3100 3300 30  0001 C CNN
+F 1 "VCC" H 3100 3300 30  0000 C CNN
+F 2 "" H 3100 3200 60  0000 C CNN
+F 3 "" H 3100 3200 60  0000 C CNN
+	1    3100 3200
 	-1   0    0    1
 $EndComp
